File: KICAD/BackupProjects_benedictdied_personal_0_20240606.kicad_pcb (KiCad board)
At the start: 4 copper layers, 62.5 x 43.7 mm, 56 parts, among them J2 HDR-M-2.54_1x1, Q1 AO3400A, U3 ADR5040ARTZ-REEL7_C144273, U4 MCP4822-E/SN, U5 K7803M-1000R3, U6 ESP32-WROVER-B

Commit message: Updating to latest changes from Bene
Parts:
- removed C10: 100nF, BackupProjects_benedictdied_personal_0_20240606:C0402
- removed C11: 10uF, BackupProjects_benedictdied_personal_0_20240606:C0402
- removed C12: 22uF, BackupProjects_benedictdied_personal_0_20240606:C0805
- removed C18: 10uF, BackupProjects_benedictdied_personal_0_20240606:C1206
- removed R16: 10K, BackupProjects_benedictdied_personal_0_20240606:R0402
- added D1: H3V3L10B, Diode_SMD:D_SOD-882D, F.Cu at (208.0, 120.0)
- added D2: H3V3L10B, Diode_SMD:D_SOD-882D, F.Cu at (208.0, 122.3)
- added J1: xiao_single-header-1_p1-is-p1, Connector_PinSocket_2.54mm:PinSocket_1x07_P2.54mm_Vertical, F.Cu at (204.2, 101.3)
- added J3: xiao_single-header-2_p1-is-p8, Connector_PinSocket_2.54mm:PinSocket_1x07_P2.54mm_Vertical, F.Cu at (208.8, 101.3)
- added J4: XH_to-mainboard, Connector_JST:JST_XH_B4B-XH-A_1x04_P2.50mm_Vertical, F.Cu at (214.5, 102.3)
- added J5: XH_to-mainboard, Connector_JST:JST_XH_B4B-XH-A_1x04_P2.50mm_Vertical, F.Cu at (214.5, 110.1)
- added JP1: input-12V-is-5V_NO, Jumper:SolderJumper-2_P1.3mm_Open_RoundedPad1.0x1.5mm, F.Cu at (227.7, 100.7)
- added JP2: XH-direct-gpio_SDA_NO, Jumper:SolderJumper-2_P1.3mm_Open_RoundedPad1.0x1.5mm, F.Cu at (227.7, 104.3)
- added JP3: XH-direct-gpio_SCL_NO, Jumper:SolderJumper-2_P1.3mm_Open_RoundedPad1.0x1.5mm, F.Cu at (227.7, 107.8)
- added LASER1: HDR-M-2.54_1x2, Connector_PinHeader_2.54mm:PinHeader_1x02_P2.54mm_Vertical, F.Cu at (204.2, 121.1)
- added PIN1: HDR-M-2.54_1x3, Connector_PinHeader_2.54mm:PinHeader_1x03_P2.54mm_Vertical, F.Cu at (221.8, 116.9)
- added POUT1: HDR-M-2.54_1x3, Connector_PinHeader_2.54mm:PinHeader_1x03_P2.54mm_Vertical, F.Cu at (226.5, 116.9)
- added R19: 1k, Resistor_SMD:R_0402_1005Metric, F.Cu at (208.0, 124.5)
- added U2: LM324, Package_SO:SOIC-14_3.9x8.7mm_P1.27mm, F.Cu at (215.3, 119.8)
- C1: footprint BackupProjects_benedictdied_personal_0_20240606:C0402 -> Resistor_SMD:R_0603_1608Metric
- C14, C15: footprint BackupProjects_benedictdied_personal_0_20240606:C0805 -> Resistor_SMD:R_0603_1608Metric
- C2, C5, C6, C8: footprint BackupProjects_benedictdied_personal_0_20240606:C0603 -> Resistor_SMD:R_0603_1608Metric
- C7, C9: footprint BackupProjects_benedictdied_personal_0_20240606:CAP-D10.0×F5.0 -> Capacitor_SMD:CP_Elec_10x10
- L1, L2: footprint BackupProjects_benedictdied_personal_0_20240606:IND-TH_BD10.0-P5.00-D0.7 -> Inductor_SMD:L_Neosid_SMs95_SMs95p
- LED_-15, LED_15, LED_2, LED_33, LED_5, LED_RX1, LED_TX1: footprint BackupProjects_benedictdied_personal_0_20240606:LED0603-R-RD -> LED_SMD:LED_0603_1608Metric
- Q1, U3: footprint BackupProjects_benedictdied_personal_0_20240606:SOT-23-3_L2.9-W1.6-P1.90-LS2.8-BR -> Package_TO_SOT_SMD:SOT-23-3
- R13, R14, R15: footprint BackupProjects_benedictdied_personal_0_20240606:R0603 -> Resistor_SMD:R_0603_1608Metric
- U5: value K7803M-1000R3 -> LM324; footprint BackupProjects_benedictdied_personal_0_20240606:PWRM-TH_K78XXM-1000R3 -> Package_SO:SOIC-14_3.9x8.7mm_P1.27mm
- U6: value ESP32-WROVER-B -> LM324; footprint BackupProjects_benedictdied_personal_0_20240606:WIFIM-SMD_39P-L31.4-W18.0-P1.27 -> Package_SO:SOIC-14_3.9x8.7mm_P1.27mm
Connections:
- net R14_2 renamed Net-(Q1-G)
- LED_-15 pad 1: R18_1 -> Net-(LED_-15-A)
- LED_15 pad 1: R17_1 -> Net-(LED_15-A)
- LED_2 pad 1: LED_2_1 -> Net-(LED_2-A)
- LED_33 pad 1: LED_33_1 -> Net-(LED_33-A)
- LED_5 pad 1: LED_5_1 -> Net-(LED_5-A)
- LED_RX1 pad 1: LED_RX1_1 -> Net-(LED_RX1-A)
- LED_TX1 pad 1: LED_TX1_1 -> Net-(LED_TX1-A)
- U5 pad 1: +15V -> unconnected-(U5-Pad1)
- U5 pad 3: 3.3V -> unconnected-(U5A-+-Pad3)
- U6 pad 1: GND -> VREF_B
- U6 pad 10: SDI -> Net-(U6C-+)
- U6 pad 11: SCK -> (no net)
- U6 pad 12: CS -> (no net)
- U6 pad 13: IO14 -> (no net)
- U6 pad 14: IO12 -> (no net)
- U6 pad 2: 3.3V -> VREF
- U6 pad 3: R16_1 -> VREF_B
- U6 pad 4: SENSOR_VP -> (no net)
- U6 pad 5: SENSOR_VN -> Net-(U6B-+)
- U6 pad 6: (no net) -> GND
- U6 pad 7: (no net) -> Net-(U6B-+)
- U6 pad 8: LON -> Net-(U6C-+)
- U6 pad 9: LDAC -> GND
Routing:
- net VREF: track 14.0 -> 2.37 mm, vias 0 -> 1
- net Net-(LED_33-A): track 0.00 -> 4.74 mm, vias 0 -> 1
- net Net-(Q1-G): track 2.23 -> 5.91 mm
- net LASER-: track 3.68 -> 0.00 mm
- net Net-(LED_2-A): track 0.00 -> 3.12 mm
- net Net-(LED_5-A): track 0.00 -> 3.00 mm, vias 0 -> 1
- net Net-(LED_15-A): track 0.00 -> 2.32 mm, vias 0 -> 1
- net GND: track 103.2 -> 101.7 mm, vias 36 -> 31
- net VREF_B: vias 0 -> 1
- added copper zone on B.Cu, net VREF
- removed copper zone on B.Cu, net 3.3V
