File: KICAD/_autosave-BackupProjects_benedictdied_personal_0_20240606.kicad_pcb (KiCad board)
At the start: 4 copper layers, 62.5 x 43.7 mm, 56 parts, among them J2 HDR-M-2.54_1x1, Q1 AO3400A, U3 ADR5040ARTZ-REEL7_C144273, U4 MCP4822-E/SN, U5 K7803M-1000R3, U6 ESP32-WROVER-B

Commit message: updating kicad
Parts:
- removed C10: 100nF, BackupProjects_benedictdied_personal_0_20240606:C0402
- removed C11: 10uF, BackupProjects_benedictdied_personal_0_20240606:C0402
- removed C12: 22uF, BackupProjects_benedictdied_personal_0_20240606:C0805
- removed C18: 10uF, BackupProjects_benedictdied_personal_0_20240606:C1206
- removed R16: 10K, BackupProjects_benedictdied_personal_0_20240606:R0402
- added D1: H3V3L10B, Diode_SMD:D_SOD-882D, F.Cu at (216.5, 113.7)
- added D2: H3V3L10B, Diode_SMD:D_SOD-882D, F.Cu at (216.5, 116.0)
- added J1: xiao_single-header-1_p1-is-p1, Connector_PinSocket_2.54mm:PinSocket_1x07_P2.54mm_Vertical, F.Cu at (133.1, 105.1)
- added J3: xiao_single-header-2_p1-is-p8, Connector_PinSocket_2.54mm:PinSocket_1x07_P2.54mm_Vertical, F.Cu at (116.6, 105.1)
- added J4: XH_to-mainboard, Connector_JST:JST_XH_B4B-XH-A_1x04_P2.50mm_Vertical, F.Cu at (204.1, 105.3)
- added J5: XH_to-mainboard, Connector_JST:JST_XH_B4B-XH-A_1x04_P2.50mm_Vertical, F.Cu at (204.1, 113.1)
- added JP1: input-12V-is-5V_NO, Jumper:SolderJumper-2_P1.3mm_Open_RoundedPad1.0x1.5mm, F.Cu at (217.2, 103.7)
- added JP2: XH-direct-gpio_SDA_NO, Jumper:SolderJumper-2_P1.3mm_Open_RoundedPad1.0x1.5mm, F.Cu at (217.2, 107.2)
- added JP3: XH-direct-gpio_SCL_NO, Jumper:SolderJumper-2_P1.3mm_Open_RoundedPad1.0x1.5mm, F.Cu at (217.2, 110.8)
- added LASER1: HDR-M-2.54_1x2, Connector_PinHeader_2.54mm:PinHeader_1x02_P2.54mm_Vertical, F.Cu at (181.2, 138.1)
- added PIN1: HDR-M-2.54_1x3, Connector_PinHeader_2.54mm:PinHeader_1x03_P2.54mm_Vertical, F.Cu at (171.9, 138.1)
- added POUT1: HDR-M-2.54_1x3, Connector_PinHeader_2.54mm:PinHeader_1x03_P2.54mm_Vertical, F.Cu at (176.6, 138.1)
- added R19: 1k, Resistor_SMD:R_0402_1005Metric, F.Cu at (192.4, 102.4)
- added U2: LM324, Package_SO:SOIC-14_3.9x8.7mm_P1.27mm, F.Cu at (194.1, 129.1)
- C1: footprint BackupProjects_benedictdied_personal_0_20240606:C0402 -> Resistor_SMD:R_0603_1608Metric
- C14, C15: footprint BackupProjects_benedictdied_personal_0_20240606:C0805 -> Resistor_SMD:R_0603_1608Metric
- C2, C5, C6, C8: footprint BackupProjects_benedictdied_personal_0_20240606:C0603 -> Resistor_SMD:R_0603_1608Metric
- C7, C9: footprint BackupProjects_benedictdied_personal_0_20240606:CAP-D10.0×F5.0 -> Capacitor_SMD:CP_Elec_10x10
- L1, L2: footprint BackupProjects_benedictdied_personal_0_20240606:IND-TH_BD10.0-P5.00-D0.7 -> Inductor_SMD:L_Neosid_SMs95_SMs95p
- LED_-15, LED_15, LED_2, LED_33, LED_5, LED_RX1, LED_TX1: footprint BackupProjects_benedictdied_personal_0_20240606:LED0603-R-RD -> LED_SMD:LED_0603_1608Metric
- Q1, U3: footprint BackupProjects_benedictdied_personal_0_20240606:SOT-23-3_L2.9-W1.6-P1.90-LS2.8-BR -> Package_TO_SOT_SMD:SOT-23-3
- R13, R14, R15: footprint BackupProjects_benedictdied_personal_0_20240606:R0603 -> Resistor_SMD:R_0603_1608Metric
- U5: value K7803M-1000R3 -> LM324; footprint BackupProjects_benedictdied_personal_0_20240606:PWRM-TH_K78XXM-1000R3 -> Package_SO:SOIC-14_3.9x8.7mm_P1.27mm
- U6: value ESP32-WROVER-B -> LM324; footprint BackupProjects_benedictdied_personal_0_20240606:WIFIM-SMD_39P-L31.4-W18.0-P1.27 -> Package_SO:SOIC-14_3.9x8.7mm_P1.27mm
- moved U6 81.6 mm to (210.9, 129.1), turned to 0 degrees
- moved U5 76.8 mm to (202.5, 129.1), turned to 0 degrees
Connections:
- net R14_2 renamed Net-(Q1-G)
- LED_-15 pad 1: R18_1 -> Net-(LED_-15-A)
- LED_15 pad 1: R17_1 -> Net-(LED_15-A)
- LED_2 pad 1: LED_2_1 -> Net-(LED_2-A)
- LED_33 pad 1: LED_33_1 -> Net-(LED_33-A)
- LED_5 pad 1: LED_5_1 -> Net-(LED_5-A)
- LED_RX1 pad 1: LED_RX1_1 -> Net-(LED_RX1-A)
- LED_TX1 pad 1: LED_TX1_1 -> Net-(LED_TX1-A)
- U5 pad 1: +15V -> unconnected-(U5-Pad1)
- U5 pad 3: 3.3V -> unconnected-(U5A-+-Pad3)
- U6 pad 1: GND -> VREF_B
- U6 pad 10: SDI -> Net-(U6C-+)
- U6 pad 11: SCK -> (no net)
- U6 pad 12: CS -> (no net)
- U6 pad 13: IO14 -> (no net)
- U6 pad 14: IO12 -> (no net)
- U6 pad 2: 3.3V -> VREF
- U6 pad 3: R16_1 -> VREF_B
- U6 pad 4: SENSOR_VP -> (no net)
- U6 pad 5: SENSOR_VN -> Net-(U6B-+)
- U6 pad 6: (no net) -> GND
- U6 pad 7: (no net) -> Net-(U6B-+)
- U6 pad 8: LON -> Net-(U6C-+)
- U6 pad 9: LDAC -> GND
Routing:
- net (no net): track 3.81 -> 59.7 mm, vias 9 -> 4
- net IO13: track 35.1 -> 0.00 mm, vias 1 -> 0
- net SENSOR_VN: track 34.9 -> 0.00 mm, vias 1 -> 0
- net SENSOR_VP: track 34.3 -> 0.00 mm, vias 1 -> 0
- net IO12: track 34.2 -> 0.00 mm, vias 1 -> 0
- net TX: track 34.1 -> 0.00 mm
- net GND: track 103.2 -> 69.8 mm, vias 36 -> 20
- net IO14: track 32.4 -> 0.00 mm, vias 1 -> 0
- net RX: track 26.7 -> 0.00 mm
- net Net-(LED_TX1-A): track 0.00 -> 14.9 mm
- net IO0: track 14.5 -> 0.00 mm
- net VREF: track 14.0 -> 2.37 mm
- net IO5: track 11.5 -> 0.00 mm
- net IO15: track 10.9 -> 0.00 mm, vias 1 -> 0
- net IO22: track 10.6 -> 0.00 mm
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Other:
- board text removed: "18"
- board text removed: "19"
- board text removed: "21"
- board text removed: "22"
- board text removed: "23"
- board text removed: "4"
- board text removed: "5"
