File: KICAD/_autosave-BackupProjects_benedictdied_personal_0_20240606.kicad_sch (KiCad schematic)
At the start: 69 parts, among them J2 HDR-M-2.54_1x1, Q1 AO3400A, U1.1 LM324DT, U1.2 LM324DT, U1.3 LM324DT, U1.4 LM324DT, U2.1 LM324DT, U2.2 LM324DT, U2.3 LM324DT, U2.4 LM324DT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

Commit message: updating kicad
Parts:
- removed C10: 100nF, symbol CL05B104KO5NNNC_1
- removed C11: 10uF, symbol CL05A106MQ5NUNC
- removed C12: 22uF, symbol CL21A226MAQNNNE
- removed C18: 10uF, symbol CL31A106KBHNNNE
- removed GPIO: HDR-M-2.54_1x16, symbol HDR-M-2.54_1x16
- removed PROGRAM: HDR-M-2.54_1x5, symbol HDR-M-2.54_1x5
- removed R16: 10K, symbol 0402WGF1202TCE
- removed U1.1: LM324DT, symbol LM324DT
- removed U1.2: LM324DT, symbol LM324DT_1
- removed U1.3: LM324DT, symbol LM324DT_2
- removed U1.4: LM324DT, symbol LM324DT_3
- removed U2.1: LM324DT, symbol LM324DT_4
- removed U2.2: LM324DT, symbol LM324DT_5
- removed U2.3: LM324DT, symbol LM324DT_6
- removed U2.4: LM324DT, symbol LM324DT_7
- removed U5: K7803M-1000R3, symbol K7803M-1000R3
- removed U6: ESP32-WROVER-B, symbol ESP32-WROVER-B
- added D1, D2: H3V3L10B, Diode_SMD:D_SOD-882D, symbol Device:D_TVS_Small
- added J1: xiao_single-header-1_p1-is-p1, Connector_PinSocket_2.54mm:PinSocket_1x07_P2.54mm_Vertical, symbol Connector:Conn_01x07_Socket
- added J3: xiao_single-header-2_p1-is-p8, Connector_PinSocket_2.54mm:PinSocket_1x07_P2.54mm_Vertical, symbol Connector:Conn_01x07_Socket
- added J4, J5: XH_to-mainboard, Connector_JST:JST_XH_B4B-XH-A_1x04_P2.50mm_Vertical, symbol Connector_Generic:Conn_01x04
- added JP1: input-12V-is-5V_NO, Jumper:SolderJumper-2_P1.3mm_Open_RoundedPad1.0x1.5mm, symbol Jumper:SolderJumper_2_Open
- added JP2: XH-direct-gpio_SDA_NO, Jumper:SolderJumper-2_P1.3mm_Open_RoundedPad1.0x1.5mm, symbol Jumper:SolderJumper_2_Open
- added JP3: XH-direct-gpio_SCL_NO, Jumper:SolderJumper-2_P1.3mm_Open_RoundedPad1.0x1.5mm, symbol Jumper:SolderJumper_2_Open
- added R19: 1k, Resistor_SMD:R_0402_1005Metric, symbol Device:R_Small
- added U1: xiao_esp32s3, lib:XIAO-Generic-Thruhole-14P-2.54-21X17.8MM, symbol xiao-esp32s3_lib:xiao_esp32s3
- added U2, U5, U6: LM324, Package_SO:SOIC-14_3.9x8.7mm_P1.27mm, symbol Amplifier_Operational:LM324
- C1, C14, C15, C2, C5, C6, C8, R13, R14, R15: footprint (none) -> Resistor_SMD:R_0603_1608Metric
- C7, C9: footprint (none) -> Capacitor_SMD:CP_Elec_10x10
- L1, L2: footprint (none) -> Inductor_SMD:L_Neosid_SMs95_SMs95p
- LASER: footprint (none) -> Connector_PinHeader_2.54mm:PinHeader_1x02_P2.54mm_Vertical
- LED_-15, LED_15, LED_2, LED_33, LED_5, LED_RX1, LED_TX1: footprint (none) -> LED_SMD:LED_0603_1608Metric
- PIN, POUT: footprint (none) -> Connector_PinHeader_2.54mm:PinHeader_1x03_P2.54mm_Vertical
- Q1, U3: footprint (none) -> Package_TO_SOT_SMD:SOT-23-3
Connections:
- net 3.3v: now also J3.5 (Pin_5), U1.12 (3V3)
- net CS: now also J3.4 (Pin_4), U1.11 (PA6_A10_D10_MOSI)
- net GND: now also D1.1 (A1), D2.1 (A1), J3.6 (Pin_6), J4.1 (Pin_1), J5.1 (Pin_1), U1.13 (GND), U2.13 (-), U2.2 (-), U5.2 (-), U6.6 (-), U6.9 (-)
- net L+: now also U2.7
- net L-: now also U2.14
- net LDAC: now also J1.7 (Pin_7), U1.7 (PB08_A6_TX)
- net LON: now also J3.1 (Pin_1), U1.8 (PB09_D7_RX)
- net R+: now also U2.8
- net R-: now also U2.1
- net SCK: now also J3.3 (Pin_3), U1.10 (PA5_A9_D9_MISO)
- net SDI: now also J3.2 (Pin_2), U1.9 (PA7_A8_D8_SCK)
- net VREF: now also U6.2 (-)
- net VREF_B: now also U6.1, U6.3 (+)
- net at R10.2, R9.1: now also U2.12 (+)
- net at R1.1, R4.2: now also U2.10 (+)
- net at R6.2, R7.1: now also U2.5 (+)
- net at R2.2, R3.2: now also U2.9 (-)
- net at R5.2, R8.2: now also U2.6 (-)
- net at R11.1, R12.2: now also U2.3 (+)
- new net: U6.10 (+), U6.8
- new net: J1.6 (Pin_6), J5.2 (Pin_2), U1.6 (PA9_A5_D5_SCL)
- new net: J1.5 (Pin_5), J5.3 (Pin_3), U1.5 (PA8_A4_D4_SDA)
- new net: J1.4 (Pin_4), J5.4 (Pin_4), U1.4 (PA11_A3_D3)
- new net: J1.1 (Pin_1), U1.1 (PA02_A0_D0)
- new net: U6.5 (+), U6.7
- new net +12V: J4.2 (Pin_2), JP1.1 (A)
- new net +3.3V: R19.1
- new net +5V: J3.7 (Pin_7), JP1.2 (B), U1.14 (5V)
- new net CANbus/CANbus_N: J4.4 (Pin_4), JP3.2 (B)
- new net CANbus/CANbus_P: J4.3 (Pin_3), JP2.2 (B)
- new net I2C-1_SCL: D2.2 (A2), J1.2 (Pin_2), JP3.1 (A), U1.2 (PA4_A1_D1)
- new net I2C-1_SDA: D1.2 (A2), J1.3 (Pin_3), JP2.1 (A), U1.3 (PA10_A2_D2)
- no-connect marks 11 -> 0
Other:
- added sheet CANbus (canbus.kicad_sch)
- note added: "3.3V"
- note added: "CONNECTIONS / PIN DEFINITIONS (XIAO): D0 -> pin 1 D1 -> pin 2 D2 -> pin 3 D3 -> pin 4 D4 -> pin 5 D5 -> pin 6 D6 -> pin 43 D7 -> pin 44 D8 -> pin 7 D9 -> pin 8 D10 -> pin 9 Here we map: - PIN_NUM_MISO -> -1 (not used) - PIN_NUM_SCK -> GPIO 8 (D9) - PIN_NUM_SDI -> GPIO 7 (D8) - PIN_NUM_CS -> GPIO 9 (D10) - PIN_NUM_LDAC -> GPIO 6 (D5) - PIN_NUM_LASER -> GPIO 43 (D6) - PIN_NUM_TRIG_PIXEL-> GPIO 2 (D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"
- note added: "ESP as controller"
- note added: "JSH XH THT, straight up, cable perpendicular to board cable comes out parallel to motor axis"
- note added: "Layout hint: USB port is on side of the 5V pin"
- note added: "Power budget: (OUT) 700mA @ 3.3V, (IN) 520 mA @ 5V Xiao built-in buck converter (SGM6029) efficiency: min. 90%"
- note added: "To enable I2C and disable CAN, also toggle solderjumpers and 0-resistors in CANbus sheet."
- note removed: "ESP32 Module"
- note removed: "Power Regulator"
- moved on the sheet: C2, C8, PIN, POUT, R15, U3
